File: Rev4/CAD/eagle/lvc.sch (EAGLE design)
At the start: 26 parts, among them J1 3,5MM_1X2_SCREWTERM, J2 3,5MM_1X2_SCREWTERM, Q1 SI7997DP

Commit message: Updated voltage divider resistor values
Parts:
- R10: value 301k -> 1M
- R11: value 10k -> 100k
- R7: value 1.5M -> 1M
- R8: value 510k -> 1M
Other:
- note added: "Should be RK7002BMT116"
Changed lines of the file:
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@@
 <part name="GND10" library="supply1" deviceset="GND" device=""/>
 <part name="S1" library="NR_switch" deviceset="CL-SB-13B-02" device=""/>
-<part name="R7" library="resistor" deviceset="R-US_" device="R0603" value="1.5M"/>
-<part name="R8" library="resistor" deviceset="R-US_" device="R0603" value="510k"/>
+<part name="R7" library="resistor" deviceset="R-US_" device="R0603" value="1M"/>
+<part name="R8" library="resistor" deviceset="R-US_" device="R0603" value="1M"/>
 <part name="R9" library="resistor" deviceset="R-US_" device="R0603" value="1.5M"/>
-<part name="R10" library="resistor" deviceset="R-US_" device="R0603" value="301k"/>
+<part name="R10" library="resistor" deviceset="R-US_" device="R0603" value="1M"/>
 <part name="VR1" library="NR_pot" deviceset="BOURNS_3214W" device=""/>
-<part name="R11" library="resistor" deviceset="R-US_" device="R0603" value="10k"/>
+<part name="R11" library="resistor" deviceset="R-US_" device="R0603" value="100k"/>
 <part name="GND12" library="supply1" deviceset="GND" device=""/>
 <part name="GND13" library="supply1" deviceset="GND" device=""/>
@@
 <text x="226.06" y="119.38" size="3.81" layer="97">Reverse Polarity
 Protection</text>
+<text x="78.74" y="58.42" size="1.778" layer="97">Should be RK7002BMT116</text>
 </plain>
 <instances>

Commit message: Added comparator protection; cleaned up schematic
Parts:
- added D1: BZT52B8V2, vishay1:BZT52B8V2
- R11: value 100k -> 10k
- R9: value 1.5M -> 2M
Connections:
- net N$2 renamed LED
- net GND: now also D1.A
- net V_DIV: now also D1.C
Other:
- note added: "Cutoff"
- note added: "LTST-C191KGKT"
- note removed: "Analog Buffer"
- note removed: "TPI"
- moved on the sheet: C1, C2, LED1, R1, U$1, U$2

Commit message: Added Rev4 final
Parts:
- removed R11: 10k, resistor:R-US_R0603
- removed R13: 1M, resistor:R-US_R0603
- removed U$2: TLV76033DBZR, rohm1:TLV76033DBZR
- added R5, R6: 1M, resistor:R-US_R0603
- added U1: L78L33ACUTR, LR_vreg:L78L33ACUTR
- C1: value 0.1uF -> 0.33uF
- C2: value 0.33uF -> 0.1uF
- R7: value 1M -> 2M
- R9: value 2M -> 10k
Connections:
- net 2_CELL: now also R5.2, R6.1; no longer R7.2, R8.1
- net 3_CELL: now also R7.2, R8.1; no longer R10.1, R9.2
- net EN: now also R5.1; no longer R11.1
- net GND: now also R6.2, U1.GND; no longer R13.2, U$2.GND
- net LED: now also C2.1, U1.VOUT; no longer C1.1, U$2.OUT
- net N$11: now also R9.2; no longer R11.2
- net N$6: now also R10.1; no longer R13.1
- net VOUT: now also C1.1, U1.VIN; no longer C2.1, U$2.VIN
Other:
- note added: "C1 rated to at least 35 V"
- note added: "NOTE: All resistors +/- 1.0% tolerance All capacitors +/- 10% tolerance"
- note added: "R3 rated to at least 0.2 W"
- moved on the sheet: C1, C2, R10, R7, R8, R9
