File: Rev6/CAD/eagle/lvc.sch (EAGLE design)
At the start: 31 parts, among them J1 3,5MM_1X2_SCREWTERM, J2 3,5MM_1X2_SCREWTERM, Q1 SI7997DP, U1 L78L33ACUTR, U2 TLV170IDBVR

Commit message: Updated buffer to be upstream of comparator
Parts:
- C3: value 0.33uF -> 50pF
- R11: value 3k -> 100k; device resistor:R-US_R0603 -> rcl:R-US_R0603
Connections:
- removed net CUTOFF: U$1.!RST!, U2.+IN
- removed net N$1: R11.1, U2.-IN, U2.OUT
- new net V_DIV_BUF: C3.1, R11.2, U$1.VCC, U2.-IN, U2.OUT
- net GND: now also R11.1
- net LOAD: now also U$1.!RST!; no longer C3.1, R11.2
- net V_DIV: now also U2.+IN; no longer U$1.VCC
Other:
- moved on the sheet: C3, R11, U$1
Changed lines of the file:
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@@
 <part name="P+1" library="supply1" library_urn="urn:adsk.eagle:library:371" deviceset="V+" device=""/>
 <part name="GND5" library="supply1" library_urn="urn:adsk.eagle:library:371" deviceset="GND" device=""/>
-<part name="R11" library="resistor" library_urn="urn:adsk.eagle:library:348" deviceset="R-US_" device="R0603" package3d_urn="urn:adsk.eagle:package:26057/1" value="3k"/>
-<part name="C3" library="rcl" library_urn="urn:adsk.eagle:library:334" deviceset="C-US" device="C0603" package3d_urn="urn:adsk.eagle:package:23616/2" value="0.33uF"/>
-<part name="GND6" library="supply1" library_urn="urn:adsk.eagle:library:371" deviceset="GND" device=""/>
 <part name="GND11" library="supply1" library_urn="urn:adsk.eagle:library:371" deviceset="GND" device=""/>
 <part name="C4" library="rcl" library_urn="urn:adsk.eagle:library:334" deviceset="C-US" device="C0603" package3d_urn="urn:adsk.eagle:package:23616/2" value="0.1uF"/>
+<part name="R11" library="rcl" library_urn="urn:adsk.eagle:library:334" deviceset="R-US_" device="R0603" package3d_urn="urn:adsk.eagle:package:23555/2" value="100k"/>
+<part name="GND6" library="supply1" library_urn="urn:adsk.eagle:library:371" deviceset="GND" device=""/>
+<part name="C3" library="rcl" library_urn="urn:adsk.eagle:library:334" deviceset="C-US" device="C0603" package3d_urn="urn:adsk.eagle:package:23616/2" value="50pF"/>
+<part name="GND15" library="supply1" library_urn="urn:adsk.eagle:library:371" deviceset="GND" device=""/>
 </parts>
 <sheets>
@@
 <attribute name="NAME" x="68.58" y="99.06" size="2.54" layer="95"/>
 </instance>
-<instance part="U$1" gate="G$1" x="106.68" y="177.8"/>
-<instance part="GND1" gate="1" x="88.9" y="165.1"/>
+<instance part="U$1" gate="G$1" x="111.76" y="172.72"/>
+<instance part="GND1" gate="1" x="93.98" y="160.02"/>
 <instance part="U$3" gate="G$1" x="48.26" y="55.88"/>
 <instance part="C2" gate="G$1" x="63.5" y="172.72"/>
@@
 </instance>
 <instance part="GND5" gate="1" x="124.46" y="78.74"/>
-<instance part="R11" gate="G$1" x="142.24" y="91.44" smashed="yes">
-<attribute name="NAME" x="138.43" y="87.8586" size="1.778" layer="95"/>
-<attribute name="VALUE" x="138.43" y="85.598" size="1.778" layer="96"/>
-</instance>
-<instance part="C3" gate="G$1" x="149.86" y="86.36"/>
-<instance part="GND6" gate="1" x="149.86" y="73.66"/>
 <instance part="GND11" gate="1" x="137.16" y="101.6"/>
 <instance part="C4" gate="G$1" x="137.16" y="111.76"/>
+<instance part="R11" gate="G$1" x="114.3" y="66.04" rot="R90"/>
+<instance part="GND6" gate="1" x="147.32" y="76.2"/>
+<instance part="C3" gate="G$1" x="147.32" y="86.36"/>
+<instance part="GND15" gate="1" x="114.3" y="55.88"/>
 </instances>
 <busses>
@@
 <pinref part="U$1" gate="G$1" pin="GND"/>
 <pinref part="GND1" gate="1" pin="GND"/>
-<wire x1="93.98" y1="172.72" x2="88.9" y2="172.72" width="0.1524" layer="91"/>
-<wire x1="88.9" y1="172.72" x2="88.9" y2="167.64" width="0.1524" layer="91"/>
+<wire x1="99.06" y1="167.64" x2="93.98" y2="167.64" width="0.1524" layer="91"/>
+<wire x1="93.98" y1="167.64" x2="93.98" y2="162.56" width="0.1524" layer="91"/>
 </segment>
 <segment>
@@
 </segment>
 <segment>
-<pinref part="C3" gate="G$1" pin="2"/>
-<pinref part="GND6" gate="1" pin="GND"/>
-<wire x1="149.86" y1="81.28" x2="149.86" y2="76.2" width="0.1524" layer="91"/>
-</segment>
-<segment>
 <pinref part="C4" gate="G$1" pin="2"/>
 <pinref part="GND11" gate="1" pin="GND"/>
 <wire x1="137.16" y1="106.68" x2="137.16" y2="104.14" width="0.1524" layer="91"/>
+</segment>
+<segment>
+<pinref part="GND15" gate="1" pin="GND"/>
+<pinref part="R11" gate="G$1" pin="1"/>
+<wire x1="114.3" y1="60.96" x2="114.3" y2="58.42" width="0.1524" layer="91"/>
+</segment>
+<segment>
+<pinref part="GND6" gate="1" pin="GND"/>
+<pinref part="C3" gate="G$1" pin="2"/>
+<wire x1="147.32" y1="81.28" x2="147.32" y2="78.74" width="0.1524" layer="91"/>
 </segment>
 </net>
@@
 </segment>
 <segment>
-<pinref part="R11" gate="G$1" pin="2"/>
-<wire x1="147.32" y1="91.44" x2="149.86" y2="91.44" width="0.1524" layer="91"/>
-<wire x1="154.94" y1="91.44" x2="149.86" y2="91.44" width="0.1524" layer="91"/>
-<wire x1="149.86" y1="91.44" x2="149.86" y2="88.9" width="0.1524" layer="91"/>
-<junction x="149.86" y="91.44"/>
-<pinref part="C3" gate="G$1" pin="1"/>
-<label x="154.94" y="91.44" size="1.778" layer="95" xref="yes"/>
+<pinref part="U$1" gate="G$1" pin="!RST!"/>
+<wire x1="124.46" y1="172.72" x2="129.54" y2="172.72" width="0.1524" layer="91"/>
+<label x="129.54" y="172.72" size="1.778" layer="95" xref="yes"/>
 </segment>
 </net>
@@
 </segment>
 <segment>
-<pinref part="U$1" gate="G$1" pin="VCC"/>
-<wire x1="93.98" y1="182.88" x2="88.9" y2="182.88" width="0.1524" layer="91"/>
-<label x="88.9" y="182.88" size="1.778" layer="95" rot="R180" xref="yes"/>
+<pinref part="U2" gate="G$1" pin="+IN"/>
+<wire x1="116.84" y1="93.98" x2="114.3" y2="93.98" width="0.1524" layer="91"/>
+<label x="114.3" y="93.98" size="1.778" layer="95" rot="R180" xref="yes"/>
 </segment>
 </net>
@@
 </segment>
 </net>
-<net name="CUTOFF" class="0">
-<segment>
-<pinref part="U$1" gate="G$1" pin="!RST!"/>
-<wire x1="119.38" y1="177.8" x2="127" y2="177.8" width="0.1524" layer="91"/>
-<label x="127" y="177.8" size="1.778" layer="95" xref="yes"/>
-</segment>
-<segment>
-<pinref part="U2" gate="G$1" pin="+IN"/>
-<wire x1="116.84" y1="93.98" x2="114.3" y2="93.98" width="0.1524" layer="91"/>
-<label x="114.3" y="93.98" size="1.778" layer="95" rot="R180" xref="yes"/>
-</segment>
-</net>
-<net name="N$1" class="0">
-<segment>
+<net name="V_DIV_BUF" class="0">
+<segment>
+<label x="154.94" y="91.44" size="1.778" layer="95" xref="yes"/>
 <pinref part="U2" gate="G$1" pin="OUT"/>
 <wire x1="132.08" y1="91.44" x2="134.62" y2="91.44" width="0.1524" layer="91"/>
@@
 <pinref part="U2" gate="G$1" pin="-IN"/>
 <wire x1="114.3" y1="88.9" x2="116.84" y2="88.9" width="0.1524" layer="91"/>
-<wire x1="134.62" y1="91.44" x2="137.16" y2="91.44" width="0.1524" layer="91"/>
 <junction x="134.62" y="91.44"/>
-<pinref part="R11" gate="G$1" pin="1"/>
-</segment>
-</net>
+<wire x1="134.62" y1="91.44" x2="147.32" y2="91.44" width="0.1524" layer="91"/>
+<pinref part="R11" gate="G$1" pin="2"/>
+<wire x1="147.32" y1="91.44" x2="154.94" y2="91.44" width="0.1524" layer="91"/>
+<pinref part="C3" gate="G$1" pin="1"/>
+<wire x1="147.32" y1="88.9" x2="147.32" y2="91.44" width="0.1524" layer="91"/>
+<junction x="147.32" y="91.44"/>
+<wire x1="114.3" y1="71.12" x2="114.3" y2="73.66" width="0.1524" layer="91"/>
+<junction x="114.3" y="73.66"/>
+</segment>
+<segment>
+<pinref part="U$1" gate="G$1" pin="VCC"/>
+<wire x1="99.06" y1="177.8" x2="96.52" y2="177.8" width="0.1524" layer="91"/>
+<label x="96.52" y="177.8" size="1.778" layer="95" rot="R180" xref="yes"/>
+</segment>
+</net>

Commit message: Updated diode footprints
Parts:
- removed TP1: TESTPOINT, CM_test:TESTPOINT
- added TP2: TESTPOINTNOCREAM, CM_test:TESTPOINTNOCREAM
- C3: value 50pF -> 47pF
- D2, D3: value MM3Z12VC -> DZ2J120M0L; device NR_diode:MM3Z12VC -> LR_zener:DZ2J120M0L
Connections:
- net V_DIV: now also TP2.P$1; no longer TP1.P$1
Changed lines of the file:
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@@
 <part name="GND3" library="supply1" library_urn="urn:adsk.eagle:library:371" deviceset="GND" device=""/>
 <part name="R2" library="resistor" library_urn="urn:adsk.eagle:library:348" deviceset="R-US_" device="R0603" package3d_urn="urn:adsk.eagle:package:26057/1" value="100k"/>
-<part name="D2" library="NR_diode" deviceset="MM3Z12VC" device=""/>
 <part name="R3" library="resistor" library_urn="urn:adsk.eagle:library:348" deviceset="R-US_" device="R0603" package3d_urn="urn:adsk.eagle:package:26057/1" value="3k"/>
 <part name="GND7" library="supply1" library_urn="urn:adsk.eagle:library:371" deviceset="GND" device=""/>
@@
 <part name="GND14" library="supply1" library_urn="urn:adsk.eagle:library:371" deviceset="GND" device=""/>
 <part name="FRAME1" library="frames" library_urn="urn:adsk.eagle:library:229" deviceset="FRAME_A_L" device=""/>
-<part name="TP1" library="CM_test" deviceset="TESTPOINT" device=""/>
 <part name="P+12" library="supply1" library_urn="urn:adsk.eagle:library:371" deviceset="V+" device=""/>
 <part name="S2" library="AR_switches" deviceset="CL-SB-12B-02" device=""/>
@@
 <part name="VDD1" library="supply1" library_urn="urn:adsk.eagle:library:371" deviceset="VDD" device=""/>
 <part name="VDD2" library="supply1" library_urn="urn:adsk.eagle:library:371" deviceset="VDD" device=""/>
-<part name="D3" library="NR_diode" deviceset="MM3Z12VC" device=""/>
 <part name="R10" library="resistor" library_urn="urn:adsk.eagle:library:348" deviceset="R-US_" device="R0603" package3d_urn="urn:adsk.eagle:package:26057/1" value="1M"/>
 <part name="GND19" library="supply1" library_urn="urn:adsk.eagle:library:371" deviceset="GND" device=""/>
@@
 <part name="R11" library="rcl" library_urn="urn:adsk.eagle:library:334" deviceset="R-US_" device="R0603" package3d_urn="urn:adsk.eagle:package:23555/2" value="100k"/>
 <part name="GND6" library="supply1" library_urn="urn:adsk.eagle:library:371" deviceset="GND" device=""/>
-<part name="C3" library="rcl" library_urn="urn:adsk.eagle:library:334" deviceset="C-US" device="C0603" package3d_urn="urn:adsk.eagle:package:23616/2" value="50pF"/>
+<part name="C3" library="rcl" library_urn="urn:adsk.eagle:library:334" deviceset="C-US" device="C0603" package3d_urn="urn:adsk.eagle:package:23616/2" value="47pF"/>
 <part name="GND15" library="supply1" library_urn="urn:adsk.eagle:library:371" deviceset="GND" device=""/>
+<part name="TP2" library="CM_test" deviceset="TESTPOINT" device="NOCREAM"/>
+<part name="D2" library="LR_zener" deviceset="DZ2J120M0L" device=""/>
+<part name="D3" library="LR_zener" deviceset="DZ2J120M0L" device=""/>
 </parts>
 <sheets>
@@
 <attribute name="VALUE" x="46.99" y="84.582" size="1.778" layer="96" rot="R180"/>
 </instance>
-<instance part="D2" gate="G$1" x="55.88" y="88.9" rot="R90"/>
 <instance part="R3" gate="G$1" x="48.26" y="71.12" smashed="yes" rot="R270">
 <attribute name="NAME" x="46.99" y="72.1614" size="1.778" layer="95" rot="R180"/>
@@
 <instance part="FRAME1" gate="G$1" x="0" y="0"/>
 <instance part="FRAME1" gate="G$2" x="172.72" y="0"/>
-<instance part="TP1" gate="G$1" x="160.02" y="172.72"/>
 <instance part="P+12" gate="1" x="213.36" y="114.3" smashed="yes">
 <attribute name="VALUE" x="215.9" y="116.84" size="1.778" layer="96" rot="R180"/>
@@
 <attribute name="VALUE" x="241.3" y="68.58" size="1.778" layer="96" rot="R180"/>
 </instance>
-<instance part="D3" gate="G$1" x="243.84" y="93.98" rot="R180"/>
 <instance part="R10" gate="G$1" x="254" y="83.82" smashed="yes">
 <attribute name="NAME" x="250.19" y="80.2386" size="1.778" layer="95"/>
@@
 <instance part="C3" gate="G$1" x="147.32" y="86.36"/>
 <instance part="GND15" gate="1" x="114.3" y="55.88"/>
+<instance part="TP2" gate="G$1" x="160.02" y="172.72"/>
+<instance part="D2" gate="A" x="55.88" y="88.9" rot="R90"/>
+<instance part="D3" gate="A" x="243.84" y="93.98" rot="R180"/>
 </instances>
 <busses>
@@
 <wire x1="48.26" y1="91.44" x2="48.26" y2="93.98" width="0.1524" layer="91"/>
 <junction x="48.26" y="93.98"/>
-<pinref part="D2" gate="G$1" pin="C"/>
 <wire x1="55.88" y1="91.44" x2="55.88" y2="93.98" width="0.1524" layer="91"/>
 <pinref part="Q1" gate="A" pin="S"/>
 <wire x1="66.04" y1="93.98" x2="55.88" y2="93.98" width="0.1524" layer="91"/>
 <junction x="55.88" y="93.98"/>
+<pinref part="D2" gate="A" pin="C"/>
 </segment>
 <segment>
@@
 </segment>
 <segment>
-<pinref part="D3" gate="G$1" pin="C"/>
 <pinref part="Q1" gate="B" pin="S"/>
 <wire x1="241.3" y1="93.98" x2="238.76" y2="93.98" width="0.1524" layer="91"/>
@@
 <wire x1="238.76" y1="93.98" x2="228.6" y2="93.98" width="0.1524" layer="91"/>
 <junction x="238.76" y="93.98"/>
+<pinref part="D3" gate="A" pin="C"/>
 </segment>
 <segment>
@@
 <wire x1="48.26" y1="78.74" x2="55.88" y2="78.74" width="0.1524" layer="91"/>
 <wire x1="55.88" y1="78.74" x2="76.2" y2="78.74" width="0.1524" layer="91"/>
-<pinref part="D2" gate="G$1" pin="A"/>
 <wire x1="55.88" y1="83.82" x2="55.88" y2="78.74" width="0.1524" layer="91"/>
 <junction x="55.88" y="78.74"/>
@@
 <pinref part="Q1" gate="A" pin="G"/>
 <wire x1="76.2" y1="88.9" x2="76.2" y2="78.74" width="0.1524" layer="91"/>
+<pinref part="D2" gate="A" pin="A"/>
 </segment>
 </net>
@@
 <wire x1="162.56" y1="170.18" x2="160.02" y2="170.18" width="0.1524" layer="91"/>
 <label x="157.48" y="170.18" size="1.778" layer="95" rot="R180" xref="yes"/>
-<pinref part="TP1" gate="G$1" pin="P$1"/>
 <wire x1="160.02" y1="170.18" x2="157.48" y2="170.18" width="0.1524" layer="91"/>
 <wire x1="160.02" y1="172.72" x2="160.02" y2="170.18" width="0.1524" layer="91"/>
@@
 <pinref part="D1" gate="G$1" pin="C"/>
 <wire x1="160.02" y1="167.64" x2="160.02" y2="170.18" width="0.1524" layer="91"/>
+<pinref part="TP2" gate="G$1" pin="P$1"/>
 </segment>
 <segment>
@@
 <net name="N$6" class="0">
 <segment>
-<pinref part="D3" gate="G$1" pin="A"/>
 <wire x1="248.92" y1="93.98" x2="248.92" y2="83.82" width="0.1524" layer="91"/>
 <pinref part="R10" gate="G$1" pin="1"/>
@@
 <wire x1="243.84" y1="83.82" x2="248.92" y2="83.82" width="0.1524" layer="91"/>
 <junction x="248.92" y="83.82"/>
-</segment>
-</net>
+<pinref part="D3" gate="A" pin="A"/>
+</segment>
+</net>

Commit message: Cleaned up component naming on Rev 1
Parts:
- removed U$1: NCP300LSN33T1G, onsemi:NCP300LSN33T1G
- added U3: TLV170IDBVR, LR_op_amps:TLV170IDBVR
- U1: value L78L33ACUTR -> NCP300LSN33T1G; device LR_vreg:L78L33ACUTR -> onsemi:NCP300LSN33T1G
- U2: value TLV170IDBVR -> L78L33ACUTR; device LR_op_amps:TLV170IDBVR -> LR_vreg:L78L33ACUTR
- renumbered U$3 to Q2
Connections:
- net GND: now also U2.GND, U3.V-; no longer U$1.GND, U2.V-
- net LED: now also U2.VOUT; no longer U1.VOUT
- net LOAD: now also U1.!RST!; no longer U$1.!RST!
- net V+: now also U3.V+; no longer U2.V+
- net VOUT: now also U2.VIN; no longer U1.VIN
- net V_DIV: now also U3.+IN; no longer U2.+IN
- net V_DIV_BUF: now also U1.VCC, U3.-IN, U3.OUT; no longer U$1.VCC, U2.-IN, U2.OUT
Changed lines of the file:
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@@
 <part name="GND19" library="supply1" library_urn="urn:adsk.eagle:library:371" deviceset="GND" device=""/>
 <part name="Q1" library="AR_transistor" deviceset="SI7997DP" device=""/>
-<part name="U$1" library="onsemi" deviceset="NCP300LSN33T1G" device=""/>
+<part name="U1" library="onsemi" deviceset="NCP300LSN33T1G" device=""/>
 <part name="GND1" library="supply1" library_urn="urn:adsk.eagle:library:371" deviceset="GND" device=""/>
-<part name="U$3" library="rohm1" deviceset="RR7002BMT116" device=""/>
+<part name="Q2" library="rohm1" deviceset="RR7002BMT116" device=""/>
 <part name="C2" library="rcl" library_urn="urn:adsk.eagle:library:334" deviceset="C-US" device="C0603" package3d_urn="urn:adsk.eagle:package:23616/2" value="0.1uF"/>
 <part name="C1" library="rcl" library_urn="urn:adsk.eagle:library:334" deviceset="C-US" device="C0603" package3d_urn="urn:adsk.eagle:package:23616/2" value="0.33uF"/>
@@
 <part name="D1" library="vishay1" deviceset="BZT52B8V2" device=""/>
 <part name="GND4" library="supply1" library_urn="urn:adsk.eagle:library:371" deviceset="GND" device=""/>
-<part name="U1" library="LR_vreg" deviceset="L78L33ACUTR" device=""/>
-<part name="U2" library="LR_op_amps" deviceset="TLV170IDBVR" device=""/>
+<part name="U2" library="LR_vreg" deviceset="L78L33ACUTR" device=""/>
+<part name="U3" library="LR_op_amps" deviceset="TLV170IDBVR" device=""/>
 <part name="P+1" library="supply1" library_urn="urn:adsk.eagle:library:371" deviceset="V+" device=""/>
 <part name="GND5" library="supply1" library_urn="urn:adsk.eagle:library:371" deviceset="GND" device=""/>
@@
 <attribute name="NAME" x="68.58" y="99.06" size="2.54" layer="95"/>
 </instance>
-<instance part="U$1" gate="G$1" x="111.76" y="172.72"/>
+<instance part="U1" gate="G$1" x="111.76" y="172.72"/>
 <instance part="GND1" gate="1" x="93.98" y="160.02"/>
-<instance part="U$3" gate="G$1" x="48.26" y="55.88"/>
+<instance part="Q2" gate="G$1" x="48.26" y="55.88"/>
 <instance part="C2" gate="G$1" x="63.5" y="172.72"/>
 <instance part="C1" gate="G$1" x="20.32" y="175.26"/>
@@
 <instance part="D1" gate="G$1" x="160.02" y="165.1" rot="R90"/>
 <instance part="GND4" gate="1" x="160.02" y="154.94"/>
-<instance part="U1" gate="A" x="30.48" y="180.34"/>
-<instance part="U2" gate="G$1" x="124.46" y="91.44" smashed="yes">
+<instance part="U2" gate="A" x="30.48" y="180.34"/>
+<instance part="U3" gate="G$1" x="124.46" y="91.44" smashed="yes">
 <attribute name="NAME" x="127" y="86.995" size="1.778" layer="95"/>
 <attribute name="VALUE" x="127" y="93.98" size="1.778" layer="96"/>
@@
 <pinref part="GND7" gate="1" pin="GND"/>
 <wire x1="48.26" y1="50.8" x2="48.26" y2="38.1" width="0.1524" layer="91"/>
-<pinref part="U$3" gate="G$1" pin="S"/>
+<pinref part="Q2" gate="G$1" pin="S"/>
 </segment>
 <segment>
@@
 </segment>
 <segment>
-<pinref part="U$1" gate="G$1" pin="GND"/>
+<pinref part="U1" gate="G$1" pin="GND"/>
 <pinref part="GND1" gate="1" pin="GND"/>
 <wire x1="99.06" y1="167.64" x2="93.98" y2="167.64" width="0.1524" layer="91"/>
@@
 <wire x1="63.5" y1="165.1" x2="30.48" y2="165.1" width="0.1524" layer="91"/>
 <junction x="30.48" y="165.1"/>
-<pinref part="U1" gate="A" pin="GND"/>
+<pinref part="U2" gate="A" pin="GND"/>
 </segment>
 <segment>
@@
 </segment>
 <segment>
-<pinref part="U2" gate="G$1" pin="V-"/>
+<pinref part="U3" gate="G$1" pin="V-"/>
 <pinref part="GND5" gate="1" pin="GND"/>
 <wire x1="124.46" y1="83.82" x2="124.46" y2="81.28" width="0.1524" layer="91"/>
@@
 </segment>
 <segment>
-<pinref part="U2" gate="G$1" pin="V+"/>
+<pinref part="U3" gate="G$1" pin="V+"/>
 <pinref part="P+1" gate="1" pin="V+"/>
 <wire x1="124.46" y1="99.06" x2="124.46" y2="116.84" width="0.1524" layer="91"/>
@@
 <label x="38.1" y="53.34" size="1.778" layer="95" rot="R180" xref="yes"/>
 <pinref part="R4" gate="G$1" pin="1"/>
-<pinref part="U$3" gate="G$1" pin="G"/>
-</segment>
-<segment>
-<pinref part="U$1" gate="G$1" pin="!RST!"/>
+<pinref part="Q2" gate="G$1" pin="G"/>
+</segment>
+<segment>
+<pinref part="U1" gate="G$1" pin="!RST!"/>
 <wire x1="124.46" y1="172.72" x2="129.54" y2="172.72" width="0.1524" layer="91"/>
 <label x="129.54" y="172.72" size="1.778" layer="95" xref="yes"/>
@@
 <pinref part="R3" gate="G$1" pin="2"/>
 <wire x1="48.26" y1="66.04" x2="48.26" y2="60.96" width="0.1524" layer="91"/>
-<pinref part="U$3" gate="G$1" pin="D"/>
+<pinref part="Q2" gate="G$1" pin="D"/>
 </segment>
 </net>
@@
 <wire x1="20.32" y1="180.34" x2="17.78" y2="180.34" width="0.1524" layer="91"/>
 <label x="17.78" y="180.34" size="1.778" layer="95" rot="R180" xref="yes"/>
-<pinref part="U1" gate="A" pin="VIN"/>
+<pinref part="U2" gate="A" pin="VIN"/>
 </segment>
 </net>
@@
 </segment>
 <segment>
-<pinref part="U2" gate="G$1" pin="+IN"/>
+<pinref part="U3" gate="G$1" pin="+IN"/>
 <wire x1="116.84" y1="93.98" x2="114.3" y2="93.98" width="0.1524" layer="91"/>
 <label x="114.3" y="93.98" size="1.778" layer="95" rot="R180" xref="yes"/>
@@
 <wire x1="60.96" y1="177.8" x2="63.5" y2="177.8" width="0.1524" layer="91"/>
 <label x="66.04" y="177.8" size="1.778" layer="95" xref="yes"/>
-<pinref part="U1" gate="A" pin="VOUT"/>
+<pinref part="U2" gate="A" pin="VOUT"/>
 <wire x1="63.5" y1="177.8" x2="66.04" y2="177.8" width="0.1524" layer="91"/>
 <wire x1="63.5" y1="175.26" x2="63.5" y2="177.8" width="0.1524" layer="91"/>
@@
 <segment>
 <label x="154.94" y="91.44" size="1.778" layer="95" xref="yes"/>
-<pinref part="U2" gate="G$1" pin="OUT"/>
+<pinref part="U3" gate="G$1" pin="OUT"/>
 <wire x1="132.08" y1="91.44" x2="134.62" y2="91.44" width="0.1524" layer="91"/>
 <wire x1="134.62" y1="91.44" x2="134.62" y2="73.66" width="0.1524" layer="91"/>
 <wire x1="134.62" y1="73.66" x2="114.3" y2="73.66" width="0.1524" layer="91"/>
 <wire x1="114.3" y1="73.66" x2="114.3" y2="88.9" width="0.1524" layer="91"/>
-<pinref part="U2" gate="G$1" pin="-IN"/>
+<pinref part="U3" gate="G$1" pin="-IN"/>
 <wire x1="114.3" y1="88.9" x2="116.84" y2="88.9" width="0.1524" layer="91"/>
 <junction x="134.62" y="91.44"/>
@@
 </segment>
 <segment>
-<pinref part="U$1" gate="G$1" pin="VCC"/>
+<pinref part="U1" gate="G$1" pin="VCC"/>
 <wire x1="99.06" y1="177.8" x2="96.52" y2="177.8" width="0.1524" layer="91"/>
 <label x="96.52" y="177.8" size="1.778" layer="95" rot="R180" xref="yes"/>
